Commit message: set URDF in the right config

File: examples/h1v2/urdf/h1_2_handless.urdf (robot description, URDF)
Before this commit: robot h1_2, 28 links, 27 joints
Links:
- added link world
Joints:
- added joint fixed_base_joint: type fixed, parent world, child pelvis, origin xyz=0 0 0.2 rpy=0 -1.57 0

Commit message: first TLS identif

File: examples/h1v2/urdf/h1_2_handless.urdf (robot description, URDF)
Before this commit: robot h1_2, 29 links, 28 joints
Joints:
- joint left_ankle_pitch_joint: type revolute -> fixed
- joint left_ankle_roll_joint: type revolute -> fixed
- joint left_hip_pitch_joint: type revolute -> fixed
- joint left_hip_roll_joint: type revolute -> fixed
- joint left_hip_yaw_joint: type revolute -> fixed
- joint left_knee_joint: type revolute -> fixed
- joint right_ankle_pitch_joint: type revolute -> fixed
- joint right_ankle_roll_joint: type revolute -> fixed
- joint right_elbow_joint: type revolute -> fixed
- joint right_hip_pitch_joint: type revolute -> fixed
- joint right_hip_roll_joint: type revolute -> fixed
- joint right_hip_yaw_joint: type revolute -> fixed
- joint right_knee_joint: type revolute -> fixed
- joint right_shoulder_pitch_joint: type revolute -> fixed
- joint right_shoulder_roll_joint: type revolute -> fixed
- joint right_shoulder_yaw_joint: type revolute -> fixed
- joint right_wrist_pitch_joint: type revolute -> fixed
- joint right_wrist_roll_joint: type revolute -> fixed
- joint right_wrist_yaw_joint: type revolute -> fixed
- joint torso_joint: type revolute -> fixed

Commit message: TLS almost working with mujoco data

File: examples/h1v2/urdf/h1_2_handless.urdf (robot description, URDF)
Before this commit: robot h1_2, 29 links, 28 joints
Joints:
- joint left_wrist_pitch_joint: type revolute -> fixed
- joint left_wrist_roll_joint: type revolute -> fixed
- joint left_wrist_yaw_joint: type revolute -> fixed

Commit message: update repo to identify directly in standard parameters with LMI

File: examples/h1v2/urdf/h1_2_handless.urdf (robot description, URDF)
Before this commit: robot h1_2, 29 links, 28 joints
Links:
- removed link left_ankle_pitch_link
- removed link left_ankle_roll_link
- removed link left_hip_pitch_link
- removed link left_hip_roll_link
- removed link left_hip_yaw_link
- removed link left_knee_link
- removed link pelvis
- removed link right_ankle_pitch_link
- removed link right_ankle_roll_link
- removed link right_elbow_link
- removed link right_hip_pitch_link
- removed link right_hip_roll_link
- removed link right_hip_yaw_link
- removed link right_knee_link
- removed link right_shoulder_pitch_link
- removed link right_shoulder_roll_link
- removed link right_shoulder_yaw_link
- removed link right_wrist_pitch_link
- removed link right_wrist_roll_link
- removed link right_wrist_yaw_link
Joints:
- removed joint left_ankle_pitch_joint
- removed joint left_ankle_roll_joint
- removed joint left_hip_pitch_joint
- removed joint left_hip_roll_joint
- removed joint left_hip_yaw_joint
- removed joint left_knee_joint
- removed joint right_ankle_pitch_joint
- removed joint right_ankle_roll_joint
- removed joint right_elbow_joint
- removed joint right_hip_pitch_joint
- removed joint right_hip_roll_joint
- removed joint right_hip_yaw_joint
- removed joint right_knee_joint
- removed joint right_shoulder_pitch_joint
- removed joint right_shoulder_roll_joint
- removed joint right_shoulder_yaw_joint
- removed joint right_wrist_pitch_joint
- removed joint right_wrist_roll_joint
- removed joint right_wrist_yaw_joint
- removed joint torso_joint
- joint fixed_base_joint: child pelvis -> torso_link
- joint left_wrist_pitch_joint: type fixed -> revolute
- joint left_wrist_roll_joint: type fixed -> revolute
- joint left_wrist_yaw_joint: type fixed -> revolute
